Commit message: Fixed Initial and Collisions

File: robot.urdf (robot description, URDF)
Before this commit: robot quadruped, 17 links, 16 joints
Links:
- link base_link: mass 3.17368e-05 -> 0.5; geometry collision box size=0.08 0.08 0.03; visual mesh filename=meshes/base_body.stl scale=1 1 1
- link femur_FL: mass 5.32199e-06 -> 0.02
- link femur_FR: mass 5.32199e-06 -> 0.02
- link femur_RL: mass 5.32199e-06 -> 0.02
- link femur_RR: mass 5.32199e-06 -> 0.02
- link foot_FL: mass 6.69805e-06 -> 0.01; geometry collision cylinder length=0.07 radius=0.007; visual mesh filename=meshes/leg.stl scale=1 1 1
- link foot_FR: mass 6.69805e-06 -> 0.01; geometry collision cylinder length=0.07 radius=0.007; visual mesh filename=meshes/leg.stl scale=1 1 1
- link foot_RL: mass 6.69805e-06 -> 0.01; geometry collision cylinder length=0.07 radius=0.007; visual mesh filename=meshes/leg.stl scale=1 1 1
- link foot_RR: mass 6.69805e-06 -> 0.01; geometry collision cylinder length=0.07 radius=0.007; visual mesh filename=meshes/leg.stl scale=1 1 1
- link lower_leg_FL: mass 0.0529214 -> 0.01
- link lower_leg_FR: mass 0.0529214 -> 0.03
- link lower_leg_RL: mass 0.0529214 -> 0.03
- link lower_leg_RR: mass 0.0529214 -> 0.03
- link shoulder_FL: mass 0.0529214 -> 0.05
- link shoulder_FR: mass 0.0529214 -> 0.05

Commit message: Changed the robot collision

File: robot.urdf (robot description, URDF)
Before this commit: robot quadruped, 17 links, 16 joints
Links:
- link foot_FL: geometry collision cylinder length=0.07 radius=0.01007; visual mesh filename=meshes/leg.stl scale=1 1 1
- link foot_FR: geometry collision cylinder length=0.07 radius=0.01007; visual mesh filename=meshes/leg.stl scale=1 1 1
- link foot_RL: geometry collision cylinder length=0.07 radius=0.01007; visual mesh filename=meshes/leg.stl scale=1 1 1
- link foot_RR: geometry collision cylinder length=0.07 radius=0.01007; visual mesh filename=meshes/leg.stl scale=1 1 1
